File: Eagle/old/µECU-CAN-Adapter_Verteilte_Systeme_27_09_22.brd (EAGLE design)
At the start: 80 x 63.8 mm, 21 parts, among them IC1 MCP2515, IC2 PCA82C251, Q1 16MHz

Commit message: commit all
Parts:
- added R3: 10k, rcl:R0805
- moved SV1 35.7 mm to (26.4, 6.67), turned to 0 degrees
- moved R2 34.9 mm to (1.59, -10.2), turned to 0 degrees
- moved R1 25.8 mm to (1.59, -4.13), turned to 0 degrees
- moved U$1 23.4 mm to (53.7, 22.2), turned to 0 degrees
- moved R9 23.0 mm to (53.0, 51.8), turned to 270 degrees
- moved C3 17.1 mm to (15.2, 47.3)
- moved JP2 17.0 mm to (16.8, 13.7)
- moved IC2 16.6 mm to (50.5, 42.9), turned to 270 degrees
- moved C7 16.1 mm to (23.8, 41.0), turned to 270 degrees
- moved R8 15.0 mm to (15.9, 42.2), turned to 270 degrees
- moved C6 13.3 mm to (44.5, 39.1)
- moved C5 11.7 mm to (49.2, 61.0)
- moved Q1 9.80 mm to (41.9, 57.1), turned to 90 degrees
- moved R10 9.26 mm to (63.2, 50.2), turned to 0 degrees
- moved IC1 8.47 mm to (28.6, 50.5), turned to 90 degrees
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Connections:
- net +5V: now also R3.2
- net PB1: now also LED12.2
- net PD2: now also R3.1, U$1.3; no longer LED12.2
Routing:
- net +5V: track 111.9 -> 0.00 mm
- net PB4: track 56.4 -> 0.00 mm, vias 1 -> 0
- net PB5: track 51.1 -> 0.00 mm, vias 1 -> 0
- net PB2: track 46.1 -> 0.00 mm, vias 1 -> 0
- net N$8: track 43.8 -> 0.00 mm, vias 1 -> 0
- net PB3: track 43.2 -> 0.00 mm, vias 1 -> 0
- net N$10: track 41.3 -> 0.00 mm, vias 1 -> 0
- net PC4: track 34.2 -> 0.00 mm, vias 1 -> 0
- net PD2: track 29.6 -> 0.00 mm, vias 1 -> 0
- net PC5: track 24.0 -> 0.00 mm, vias 1 -> 0
- net N$4: track 20.3 -> 0.00 mm
- net N$3: track 16.9 -> 0.00 mm
- net N$6: track 13.0 -> 0.00 mm
- net N$2: track 13.0 -> 0.00 mm
- net PD6: track 9.97 -> 0.00 mm
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