File: Eagle/old/µECU-CAN-Adapter_Verteilte_Systeme_27_09_22.sch (EAGLE design)
At the start: 21 parts, among them IC1 MCP2515, IC2 PCA82C251, Q1 16MHz

Commit message: commit all
Parts:
- added R3: 10k, rcl:R-EU_R0805
Connections:
- net +5V: now also R3.2
- net PB1: now also LED12.DIN
- net PD2: now also R3.1, U$1.ALRT; no longer LED12.DIN
Changed lines of the file:
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@@
 <setting verticaltext="up"/>
 </settings>
-<grid distance="0.1" unitdist="inch" unit="inch" style="lines" multiple="1" display="no" altdistance="0.01" altunitdist="inch" altunit="inch"/>
+<grid distance="0.0125" unitdist="inch" unit="inch" style="lines" multiple="1" display="no" altdistance="0.01" altunitdist="inch" altunit="inch"/>
 <layers>
 <layer number="1" name="Top" color="4" fill="1" visible="no" active="no"/>
@@
 <part name="R1" library="rcl" deviceset="R-EU_" device="R0805" value="10k"/>
 <part name="R2" library="rcl" deviceset="R-EU_" device="R0805" value="10k"/>
+<part name="R3" library="rcl" deviceset="R-EU_" device="R0805" value="10k"/>
 </parts>
 <sheets>
@@
 <attribute name="VALUE" x="215.265" y="145.542" size="1.778" layer="96" rot="R180"/>
 </instance>
+<instance part="R3" gate="G$1" x="248.285" y="148.59" smashed="yes" rot="R90">
+<attribute name="NAME" x="248.285" y="153.4414" size="1.778" layer="95" rot="R180"/>
+<attribute name="VALUE" x="253.365" y="144.907" size="1.778" layer="96" rot="R180"/>
+</instance>
 </instances>
 <busses>
@@
 <pinref part="U$1" gate="G$1" pin="VCC"/>
 <wire x1="231.4575" y1="154.6225" x2="231.4575" y2="156.5275" width="0.1524" layer="91"/>
+<pinref part="R3" gate="G$1" pin="2"/>
 <wire x1="231.4575" y1="156.5275" x2="231.4575" y2="157.48" width="0.1524" layer="91"/>
+<wire x1="231.4575" y1="156.5275" x2="248.285" y2="156.5275" width="0.1524" layer="91"/>
+<wire x1="248.285" y1="156.5275" x2="248.285" y2="153.67" width="0.1524" layer="91"/>
 <junction x="231.4575" y="156.5275"/>
 <pinref part="R1" gate="G$1" pin="2"/>
@@
 <pinref part="SV2" gate="G$1" pin="28"/>
 </segment>
+<segment>
+<wire x1="157.48" y1="115.2525" x2="162.56" y2="115.2525" width="0.1524" layer="91"/>
+<label x="157.48" y="115.2525" size="1.778" layer="95" rot="R180" xref="yes"/>
+<pinref part="LED12" gate="G$1" pin="DIN"/>
+</segment>
 </net>
 <net name="PD2" class="0">
@@
 </segment>
 <segment>
-<wire x1="157.48" y1="115.2525" x2="162.56" y2="115.2525" width="0.1524" layer="91"/>
-<label x="157.48" y="115.2525" size="1.778" layer="95" rot="R180" xref="yes"/>
-<pinref part="LED12" gate="G$1" pin="DIN"/>
-</segment>
-</net>
+<pinref part="U$1" gate="G$1" pin="ALRT"/>
+<wire x1="244.1575" y1="141.9225" x2="248.285" y2="141.9225" width="0.1524" layer="91"/>
+<label x="252.73" y="141.9225" size="1.778" layer="95" xref="yes"/>
+<pinref part="R3" gate="G$1" pin="1"/>
+<wire x1="248.285" y1="141.9225" x2="252.73" y2="141.9225" width="0.1524" layer="91"/>
+<wire x1="248.285" y1="143.51" x2="248.285" y2="141.9225" width="0.1524" layer="91"/>
+<junction x="248.285" y="141.9225"/>
+</segment>
+</net>
